File: mm_motor.kicad_sch (KiCad schematic)
At the start: 1 part, among them M1 N20_encoder

Commit message: tp2
Parts:
- added C11: 2.2uF, Capacitor_SMD:C_0603_1608Metric, symbol Device:C
- added C13: 0.1uF, Capacitor_SMD:C_0603_1608Metric, symbol Device:C
- added J2: Conn_01x06_Pin, Connector_PinHeader_2.54mm:PinHeader_1x06_P2.54mm_Vertical, symbol Connector:Conn_01x06_Pin
Connections:
- net C1: now also J2.3 (Pin_3)
- net C2: now also J2.4 (Pin_4)
- net MA: now also J2.1 (Pin_1)
- net MB: now also J2.6 (Pin_6)
- new net +BATT: C11.1, C13.1, J2.5 (Pin_5)
- new net GND: C11.2, C13.2, J2.2 (Pin_2)
Changed lines of the file:
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@@
 (kicad_sch (version 20230121) (generator eeschema)
   (paper "A4")
-  (hierarchical_label "C1" (shape output) (at 118.11 91.44 180) (fields_autoplaced)
-    (effects (font (size 1.27 1.27)) (justify right))
-  )
-  (hierarchical_label "C2" (shape output) (at 118.11 93.98 180) (fields_autoplaced)
-    (effects (font (size 1.27 1.27)) (justify right))
-  )
-  (hierarchical_label "MB" (shape passive) (at 118.11 99.06 180) (fields_autoplaced)
-    (effects (font (size 1.27 1.27)) (justify right))
-  )
-  (hierarchical_label "MA" (shape passive) (at 118.11 86.36 180) (fields_autoplaced)
-    (effects (font (size 1.27 1.27)) (justify right))
+  (junction (at 167.64 96.52) (diameter 0) (color 0 0 0 0)
+  )
+  (junction (at 166.37 107.95) (diameter 0) (color 0 0 0 0)
+  )
+  (junction (at 166.37 96.52) (diameter 0) (color 0 0 0 0)
+  )
+  (wire (pts (xy 167.64 96.52) (xy 179.07 96.52))
+    (stroke (width 0) (type default))
+  )
+  (wire (pts (xy 140.97 91.44) (xy 158.75 91.44))
+    (stroke (width 0) (type default))
+  )
+  (wire (pts (xy 179.07 106.68) (xy 179.07 107.95))
+    (stroke (width 0) (type default))
+  )
+  (wire (pts (xy 179.07 107.95) (xy 166.37 107.95))
+    (stroke (width 0) (type default))
+  )
+  (wire (pts (xy 140.97 86.36) (xy 157.48 86.36))
+    (stroke (width 0) (type default))
+  )
+  (wire (pts (xy 140.97 88.9) (xy 182.88 88.9))
+    (stroke (width 0) (type default))
+  )
+  (wire (pts (xy 140.97 99.06) (xy 157.48 99.06))
+    (stroke (width 0) (type default))
+  )
+  (wire (pts (xy 140.97 93.98) (xy 158.75 93.98))
+    (stroke (width 0) (type default))
+  )
+  (wire (pts (xy 166.37 96.52) (xy 167.64 96.52))
+    (stroke (width 0) (type default))
+  )
+  (wire (pts (xy 166.37 96.52) (xy 166.37 99.06))
+    (stroke (width 0) (type default))
+  )
+  (wire (pts (xy 179.07 99.06) (xy 179.07 96.52))
+    (stroke (width 0) (type default))
+  )
+  (wire (pts (xy 166.37 106.68) (xy 166.37 107.95))
+    (stroke (width 0) (type default))
+  )
+  (wire (pts (xy 140.97 96.52) (xy 166.37 96.52))
+    (stroke (width 0) (type default))
+  )
+  (wire (pts (xy 166.37 107.95) (xy 166.37 111.76))
+    (stroke (width 0) (type default))
+  )
+  (hierarchical_label "C1" (shape output) (at 158.75 91.44 0) (fields_autoplaced)
+    (effects (font (size 1.27 1.27)) (justify left))
+  )
+  (hierarchical_label "C2" (shape output) (at 158.75 93.98 0) (fields_autoplaced)
+    (effects (font (size 1.27 1.27)) (justify left))
+  )
+  (hierarchical_label "MB" (shape passive) (at 157.48 99.06 0) (fields_autoplaced)
+    (effects (font (size 1.27 1.27)) (justify left))
+  )
+  (hierarchical_label "MA" (shape passive) (at 157.48 86.36 0) (fields_autoplaced)
+    (effects (font (size 1.27 1.27)) (justify left))
+  )
+  (symbol (lib_id "power:GND") (at 166.37 111.76 0) (unit 1)
+    (in_bom yes) (on_board yes) (dnp no) (fields_autoplaced)
+    (property "Reference" "#PWR038" (at 166.37 118.11 0)
+      (effects (font (size 1.27 1.27)) hide)
+    )
+    (property "Value" "GND" (at 166.37 116.84 0)
+      (effects (font (size 1.27 1.27)))
+    )
+    (property "Footprint" "" (at 166.37 111.76 0)
+      (effects (font (size 1.27 1.27)) hide)
+    )
+    (property "Datasheet" "" (at 166.37 111.76 0)
+      (effects (font (size 1.27 1.27)) hide)
+    )
+    (pin "1")
+    (instances
+      (project "minimouse"
+        (path "/d8fa4cba-2469-4231-847f-065b6b829f44/7f113667-692a-4f4d-b16f-621d32f3f136"
+          (reference "#PWR038") (unit 1)
+        )
+        (path "/d8fa4cba-2469-4231-847f-065b6b829f44/3975acd0-18ad-47bc-9ce1-d8c4d864aafe"
+          (reference "#PWR039") (unit 1)
+        )
+      )
+    )
+  )
+  (symbol (lib_id "Device:C") (at 179.07 102.87 0) (unit 1)
+    (in_bom yes) (on_board yes) (dnp no) (fields_autoplaced)
+    (property "Reference" "C13" (at 182.88 101.6 0)
+      (effects (font (size 1.27 1.27)) (justify left))
+    )
+    (property "Value" "0.1uF" (at 182.88 104.14 0)
+      (effects (font (size 1.27 1.27)) (justify left))
+    )
+    (property "Footprint" "Capacitor_SMD:C_0603_1608Metric" (at 180.0352 106.68 0)
+      (effects (font (size 1.27 1.27)) hide)
+    )
+    (property "Datasheet" "~" (at 179.07 102.87 0)
+      (effects (font (size 1.27 1.27)) hide)
+    )
+    (pin "2")
+    (pin "1")
+    (instances
+      (project "minimouse"
+        (path "/d8fa4cba-2469-4231-847f-065b6b829f44/3975acd0-18ad-47bc-9ce1-d8c4d864aafe"
+          (reference "C13") (unit 1)
+        )
+        (path "/d8fa4cba-2469-4231-847f-065b6b829f44/7f113667-692a-4f4d-b16f-621d32f3f136"
+          (reference "C12") (unit 1)
+        )
+      )
+    )
+  )
+  (symbol (lib_id "power:+BATT") (at 167.64 96.52 0) (unit 1)
+    (in_bom yes) (on_board yes) (dnp no) (fields_autoplaced)
+    (property "Reference" "#PWR028" (at 167.64 100.33 0)
+      (effects (font (size 1.27 1.27)) hide)
+    )
+    (property "Value" "+BATT" (at 167.64 91.44 0)
+      (effects (font (size 1.27 1.27)))
+    )
+    (property "Footprint" "" (at 167.64 96.52 0)
+      (effects (font (size 1.27 1.27)) hide)
+    )
+    (property "Datasheet" "" (at 167.64 96.52 0)
+      (effects (font (size 1.27 1.27)) hide)
+    )
+    (pin "1")
+    (instances
+      (project "minimouse"
+        (path "/d8fa4cba-2469-4231-847f-065b6b829f44/7f113667-692a-4f4d-b16f-621d32f3f136"
+          (reference "#PWR028") (unit 1)
+        )
+        (path "/d8fa4cba-2469-4231-847f-065b6b829f44/3975acd0-18ad-47bc-9ce1-d8c4d864aafe"
+          (reference "#PWR029") (unit 1)
+        )
+      )
+    )
   )
   (symbol (lib_id "minimouse:N20_w_encoder") (at 115.57 57.15 0) (unit 1)
@@
         )
       )
+    )
+  )
+  (symbol (lib_id "Connector:Conn_01x06_Pin") (at 135.89 91.44 0) (unit 1)
+    (in_bom yes) (on_board yes) (dnp no) (fields_autoplaced)
+    (property "Reference" "J2" (at 136.525 81.28 0)
+      (effects (font (size 1.27 1.27)))
+    )
+    (property "Value" "Conn_01x06_Pin" (at 136.525 83.82 0)
+      (effects (font (size 1.27 1.27)))
+    )
+    (property "Footprint" "Connector_PinHeader_2.54mm:PinHeader_1x06_P2.54mm_Vertical" (at 135.89 91.44 0)
+      (effects (font (size 1.27 1.27)) hide)
+    )
+    (property "Datasheet" "~" (at 135.89 91.44 0)
+      (effects (font (size 1.27 1.27)) hide)
+    )
+    (pin "5")
+    (pin "1")
+    (pin "6")
+    (pin "4")
+    (pin "3")
+    (pin "2")
+    (instances
+      (project "minimouse"
+        (path "/d8fa4cba-2469-4231-847f-065b6b829f44/7f113667-692a-4f4d-b16f-621d32f3f136"
+          (reference "J2") (unit 1)
+        )
+        (path "/d8fa4cba-2469-4231-847f-065b6b829f44/3975acd0-18ad-47bc-9ce1-d8c4d864aafe"
+          (reference "J3") (unit 1)
+        )
+      )
+    )
+  )
+  (symbol (lib_id "power:GND") (at 182.88 88.9 0) (unit 1)
+    (in_bom yes) (on_board yes) (dnp no) (fields_autoplaced)
+    (property "Reference" "#PWR026" (at 182.88 95.25 0)
+      (effects (font (size 1.27 1.27)) hide)
+    )
+    (property "Value" "GND" (at 182.88 93.98 0)
+      (effects (font (size 1.27 1.27)))
+    )
+    (property "Footprint" "" (at 182.88 88.9 0)
+      (effects (font (size 1.27 1.27)) hide)
+    )
+    (property "Datasheet" "" (at 182.88 88.9 0)
+      (effects (font (size 1.27 1.27)) hide)
+    )
+    (pin "1")
+    (instances
+      (project "minimouse"
+        (path "/d8fa4cba-2469-4231-847f-065b6b829f44/7f113667-692a-4f4d-b16f-621d32f3f136"
+          (reference "#PWR026") (unit 1)
+        )
+        (path "/d8fa4cba-2469-4231-847f-065b6b829f44/3975acd0-18ad-47bc-9ce1-d8c4d864aafe"
+          (reference "#PWR027") (unit 1)
+        )
+      )
+    )
+  )
+  (symbol (lib_id "Device:C") (at 166.37 102.87 0) (unit 1)
+    (in_bom yes) (on_board yes) (dnp no) (fields_autoplaced)
+    (property "Reference" "C11" (at 170.18 101.6 0)
+      (effects (font (size 1.27 1.27)) (justify left))
+    )
+    (property "Value" "2.2uF" (at 170.18 104.14 0)
+      (effects (font (size 1.27 1.27)) (justify left))
+    )
+    (property "Footprint" "Capacitor_SMD:C_0603_1608Metric" (at 167.3352 106.68 0)
+      (effects (font (size 1.27 1.27)) hide)
+    )
+    (property "Datasheet" "~" (at 166.37 102.87 0)
+      (effects (font (size 1.27 1.27)) hide)
+    )
+    (pin "2")
+    (pin "1")
+    (instances
+      (project "minimouse"
+        (path "/d8fa4cba-2469-4231-847f-065b6b829f44/3975acd0-18ad-47bc-9ce1-d8c4d864aafe"
+          (reference "C11") (unit 1)
+        )
+        (path "/d8fa4cba-2469-4231-847f-065b6b829f44/7f113667-692a-4f4d-b16f-621d32f3f136"
+          (reference "C10") (unit 1)
+        )
+      )

Commit message: TP3
Parts:
- removed C11: 2.2uF, Capacitor_SMD:C_0603_1608Metric, symbol Device:C
- added R19, R21: 100, Resistor_SMD:R_0603_1608Metric, symbol Device:R
- C13: value 0.1uF -> 2.2uF
Connections:
- net C1: now also R19.2; no longer J2.3 (Pin_3)
- net C2: now also R21.2; no longer J2.4 (Pin_4)
- new net: J2.3 (Pin_3), R19.1
- new net: J2.4 (Pin_4), R21.1
