File: mm_motor_control.kicad_sch (KiCad schematic)
At the start: 0 parts

Commit message: tp2
Parts:
- added CRCOFF: 22nF, Capacitor_SMD:C_0603_1608Metric, symbol Device:C
- added CS: 2.2uF, Capacitor_SMD:C_0603_1608Metric, symbol Device:C
- added CSPOL: 22uF, Capacitor_SMD:C_0603_1608Metric, symbol Device:C
- added CSTBY, CSTBY1: 1nF, Capacitor_SMD:C_0603_1608Metric, symbol Device:C
- added R (x2): 2.2k, Resistor_SMD:R_0603_1608Metric, symbol Device:R
- added REN, RSTBY: 18k, Resistor_SMD:R_0603_1608Metric, symbol Device:R
- added ROFF: 47k, Resistor_SMD:R_0603_1608Metric, symbol Device:R
- added Rrcoff1: 1k, Resistor_SMD:R_0603_1608Metric, symbol Device:R
- added Rsnsa, Rsnsa1: 330m, Resistor_SMD:R_0603_1608Metric, symbol Device:R
- added U2: STSPIN240, Package_DFN_QFN:VQFN-16-1EP_3x3mm_P0.5mm_EP1.8x1.8mm, symbol Driver_Motor:STSPIN240
Connections:
- net EN: now also REN.1
- net FAULT: now also CSTBY1.1, REN.2, U2.13 (EN/FLT)
- net OUT_A1: now also U2.3 (OUTA1)
- net OUT_A2: now also U2.5 (OUTA2)
- net OUT_B1: now also U2.10 (OUTB1)
- net OUT_B2: now also U2.8 (OUTB2)
- net PHASE_A: now also U2.1 (PHA)
- net PHASE_B: now also U2.15 (PHB)
- net PWM_A: now also U2.2 (PWMA)
- net PWM_B: now also U2.16 (PWMB)
- net STBY/RESET: now also CSTBY.1, RSTBY.2, U2.14 (STBY/RESET)
- new net: ROFF.1, Rrcoff1.1, U2.12 (TOFF)
- new net: R.1, R.2, U2.11 (REF)
- new net: Rsnsa.1, U2.4 (SENSEA)
- new net: Rsnsa1.1, U2.9 (SENSEB)
- new net: CRCOFF.1, Rrcoff1.2
- new net +3V3: RSTBY.1
- new net +BATT: CS.1, CSPOL.1, R.1, U2.6 (VS)
- new net GND: CRCOFF.2, CS.2, CSPOL.2, CSTBY.2, CSTBY1.2, R.2, ROFF.2, Rsnsa.2, Rsnsa1.2, U2.17 (EPAD), U2.7 (GND)

Commit message: TP3
Parts:
- removed CS: 2.2uF, Capacitor_SMD:C_0603_1608Metric, symbol Device:C
- removed CSPOL: 22uF, Capacitor_SMD:C_0603_1608Metric, symbol Device:C
- removed CSTBY: 1nF, Capacitor_SMD:C_0603_1608Metric, symbol Device:C
- removed RSTBY: 18k, Resistor_SMD:R_0603_1608Metric, symbol Device:R
- added C12: 2.2uF, Capacitor_SMD:C_0603_1608Metric, symbol Device:C
- R11: renamed from Rsnsa1; footprint Resistor_SMD:R_0603_1608Metric -> Resistor_SMD:R_2512_6332Metric
- R12: renamed from Rsnsa; footprint Resistor_SMD:R_0603_1608Metric -> Resistor_SMD:R_2512_6332Metric
- R13, R14: renamed from R; value 2.2k -> 10k
- R17: renamed from REN; value 18k -> 10k
- renumbered CRCOFF to C10, CSTBY1 to C11, Rrcoff1 to R15, ROFF to R16
Connections:
- net +BATT: now also C12.1
- net GND: now also C12.2
