File: minimouse.kicad_pcb (KiCad board)
At the start: 2 copper layers, 90 x 85 mm, 22 parts, among them J1 Conn_ARM_JTAG_SWD_10, J5 Conn_01x02, M1 N20_encoder, M2 N20_encoder, U1 STM32F030C8Tx, U4 HC-SR04

Commit message: TP3
Parts:
- added C10: 22nF, Capacitor_SMD:C_0603_1608Metric, F.Cu at (163.4, 104.9)
- added C11: 1nF, Capacitor_SMD:C_0603_1608Metric, F.Cu at (149.4, 102.2)
- added C12: 2.2uF, Capacitor_SMD:C_0603_1608Metric, F.Cu at (150.8, 112.4)
- added C13: 2.2uF, Capacitor_SMD:C_0603_1608Metric, F.Cu at (189.0, 89.6)
- added C14: 2.2uF, Capacitor_SMD:C_0603_1608Metric, F.Cu at (120.3, 89.4)
- added C15: 2.2uF, Capacitor_SMD:C_0603_1608Metric, F.Cu at (153.8, 72.0)
- added C7: 2.2uF, Capacitor_SMD:C_0603_1608Metric, F.Cu at (124.7, 78.8)
- added C8: 2.2uF, Capacitor_SMD:C_0603_1608Metric, F.Cu at (123.7, 83.8)
- added C9: 2.2uF, Capacitor_SMD:C_0603_1608Metric, F.Cu at (131.5, 83.8)
- added D1: LED, LED_SMD:LED_0603_1608Metric, F.Cu at (135.3, 86.6)
- added J2: Conn_01x06_Pin, Connector_PinHeader_2.54mm:PinHeader_1x06_P2.54mm_Vertical, F.Cu at (178.6, 93.5)
- added J3: Conn_01x06_Pin, Connector_PinHeader_2.54mm:PinHeader_1x06_P2.54mm_Vertical, F.Cu at (108.3, 93.2)
- added J4: Conn_01x04_Pin, Connector_PinHeader_2.54mm:PinHeader_1x04_P2.54mm_Vertical, F.Cu at (126.7, 74.4)
- added R10: 100, Resistor_SMD:R_0603_1608Metric, F.Cu at (121.5, 78.8)
- added R11: 330m, Resistor_SMD:R_2512_6332Metric, F.Cu at (158.2, 112.8)
- added R12: 330m, Resistor_SMD:R_2512_6332Metric, F.Cu at (142.1, 108.2)
- added R13: 10k, Resistor_SMD:R_0603_1608Metric, F.Cu at (156.4, 102.3)
- added R14: 10k, Resistor_SMD:R_0603_1608Metric, F.Cu at (153.2, 102.2)
- added R15: 1k, Resistor_SMD:R_0603_1608Metric, F.Cu at (158.1, 106.8)
- added R16: 47k, Resistor_SMD:R_0603_1608Metric, F.Cu at (158.0, 109.6)
- added R17: 10k, Resistor_SMD:R_0603_1608Metric, F.Cu at (145.1, 102.2)
- added R18: 330, Resistor_SMD:R_0603_1608Metric, F.Cu at (131.5, 86.6)
- added R19: 100, Resistor_SMD:R_0603_1608Metric, F.Cu at (183.6, 89.7)
- added R20: 100, Resistor_SMD:R_0603_1608Metric, F.Cu at (113.1, 89.4)
- added R21: 100, Resistor_SMD:R_0603_1608Metric, F.Cu at (186.1, 89.7)
- added R22: 100, Resistor_SMD:R_0603_1608Metric, F.Cu at (116.5, 89.4)
- added R23: 100, Resistor_SMD:R_0603_1608Metric, F.Cu at (148.8, 71.9)
- added U2: STSPIN240, Package_DFN_QFN:VQFN-16-1EP_3x3mm_P0.5mm_EP1.8x1.8mm, F.Cu at (150.8, 107.5)
- added U3: LP5907MFX-3.3, Package_TO_SOT_SMD:SOT-23-5, F.Cu at (127.5, 84.7)
- moved C4 20.0 mm to (148.1, 76.4), turned to 90 degrees
- moved C5 18.1 mm to (142.1, 86.8)
- moved C3 16.2 mm to (156.8, 94.4), turned to -90 degrees
- moved R9 13.2 mm to (159.4, 76.5)
- moved C1 9.36 mm to (142.2, 80.8)
- moved J1 7.84 mm to (171.7, 82.2)
- moved C6 6.29 mm to (144.2, 76.5)
- moved R8 6.19 mm to (155.4, 76.4)
- moved BOOT0 6.04 mm to (162.0, 81.8)
- moved U1 6.03 mm to (150.8, 83.6)
- moved R7 5.09 mm to (152.8, 94.4)
- moved R2 5.03 mm to (142.7, 90.4)
- moved R3 5.03 mm to (143.5, 94.4)
- moved R4 5.03 mm to (145.0, 94.4)
- moved R5 5.03 mm to (146.5, 94.4)
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Connections:
- R8 pad 1: /mcu/UART1_TX -> /external_uart/EXT_UART_RX
- U1 pad 43: /mcu/UART1_RX -> /external_uart/EXT_UART_TX
Routing:
- net Net-(U2-TOFF): track 0.00 -> 47.7 mm
- net +BATT: track 0.00 -> 28.9 mm
- net +3.3V: track 0.00 -> 20.2 mm
- net /mcu/BOOT0: track 0.00 -> 13.5 mm
- net /mcu/IN_B2: track 0.00 -> 12.1 mm
- net Net-(U2-REF): track 0.00 -> 8.67 mm
- net Net-(U1-PA3): track 0.00 -> 7.76 mm
- net Net-(U1-PA4): track 0.00 -> 7.34 mm
- net Net-(U1-PA5): track 0.00 -> 6.93 mm
- net Net-(U1-PB1): track 0.00 -> 6.51 mm
- net Net-(U1-PB0): track 0.00 -> 6.02 mm
- net Net-(U1-PB6): track 0.00 -> 5.71 mm
- net Net-(U1-PA2): track 0.00 -> 5.34 mm
- net +3V3: track 0.00 -> 5.22 mm
- net Net-(C10-Pad1): track 0.00 -> 4.48 mm
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
Commit message: tp4
Parts:
- moved J3 14.6 mm to (122.9, 93.2), turned to -90 degrees
- moved R9 11.6 mm to (147.8, 76.7)
- moved R16 8.61 mm to (158.1, 101.0), turned to 90 degrees
- moved C14 7.46 mm to (112.8, 89.8)
- moved C10 7.39 mm to (163.2, 97.5)
- moved C9 7.12 mm to (137.0, 88.2), turned to -90 degrees
- moved R14 6.61 mm to (159.7, 101.0)
- moved R17 6.57 mm to (151.5, 101.0)
- moved R15 6.14 mm to (156.2, 101.0), turned to 90 degrees
- moved C4 6.12 mm to (142.1, 77.5), turned to 180 degrees
- moved R13 5.27 mm to (161.6, 101.0), turned to -90 degrees
- moved D1 4.96 mm to (134.7, 91.5), turned to 90 degrees
- moved R20 4.82 mm to (117.9, 89.8)
- moved C11 4.61 mm to (153.9, 101.0)
- moved BOOT0 4.09 mm to (159.8, 78.3)
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Routing:
- net +BATT: track 28.9 -> 265.2 mm, vias 0 -> 2
- net +3V3: track 5.22 -> 69.1 mm
- net /external_uart/EXT_UART_RX: track 0.00 -> 60.5 mm
- net /motorA/MB: track 0.00 -> 50.6 mm
- net /motorB/MB: track 0.00 -> 47.9 mm
- net GND: track 0.00 -> 43.1 mm, vias 0 -> 27
- net /mcu/TIM2_CH2: track 0.00 -> 39.7 mm, vias 0 -> 2
- net Net-(U2-TOFF): track 47.7 -> 9.25 mm
- net /mcu/TIM3_CH2: track 0.00 -> 35.7 mm
- net /mcu/TIM3_CH1: track 0.00 -> 35.4 mm, vias 0 -> 2
- net /mcu/TIM2_CH1: track 0.00 -> 34.5 mm
- net /motorB/MA: track 0.00 -> 32.3 mm
- net /external_uart/EXT_UART_TX: track 0.77 -> 32.8 mm
- net /motorA/MA: track 0.00 -> 30.1 mm
- net +3.3V: track 20.2 -> 41.0 mm, vias 0 -> 2
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
Commit message: dernier tp
Parts:
- moved D1 11.3 mm to (130.0, 81.2), turned to 0 degrees
- moved BOOT0 8.56 mm to (152.5, 74.0)
- moved R18 6.60 mm to (132.7, 81.9), turned to 90 degrees
- moved J4 6.55 mm to (120.1, 74.3), turned to 90 degrees
- moved R4 5.34 mm to (147.2, 94.3)
- moved R10 4.68 mm to (126.2, 78.5)
- moved C6 4.27 mm to (143.3, 83.7)
- moved R8 4.12 mm to (157.3, 75.2)
- moved C9 3.95 mm to (134.9, 84.9), turned to 0 degrees
- moved C3 3.92 mm to (155.9, 90.6), turned to 0 degrees
- moved R12 3.83 mm to (142.4, 112.0), turned to -90 degrees
- moved C4 3.27 mm to (145.3, 78.1)
- moved C15 2.70 mm to (158.1, 69.2)
- moved C8 2.47 mm to (128.4, 85.2), turned to -90 degrees
- moved R11 2.39 mm to (158.5, 112.3), turned to -90 degrees
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Connections:
- C15 pad 1: +3.3V -> +BATT
- C9 pad 1: +3V3 -> +3.3V
- R18 pad 1: +3V3 -> +3.3V
- U3 pad 5: +3V3 -> +3.3V
- U4 pad 2: /mcu/OUT_B9 -> Net-(U4-TRIG)
- U4 pad 3: Net-(U4-ECHO) -> /mcu/TIM8_CH2
- U4 pad 4: +3V3 -> +BATT
Routing:
- net +3.3V: track 41.0 -> 128.2 mm
- net +BATT: track 265.2 -> 342.9 mm
- net +3V3: track 69.1 -> 0.00 mm
- net /external_uart/EXT_UART_RX: track 60.5 -> 31.3 mm, vias 0 -> 2
- net /mcu/~{RESET}: track 0.00 -> 29.2 mm, vias 0 -> 2
- net /mcu/SWO: track 0.00 -> 20.6 mm
- net /mcu/SWDCLK: track 0.00 -> 19.0 mm
- net /mcu/SWDIO: track 0.00 -> 14.6 mm
- net GND: track 43.1 -> 30.6 mm, vias 27 -> 26
- net /mcu/TIM8_CH2: track 0.00 -> 12.0 mm
- net /mcu/BOOT0: track 14.3 -> 7.48 mm
- net Net-(U1-PA4): track 11.3 -> 5.31 mm, vias 2 -> 0
- net /external_uart/EXT_UART_TX: track 32.8 -> 27.5 mm, vias 0 -> 2
- net /mcu/OUT_B9: track 7.17 -> 2.17 mm
- net Net-(U1-PB6): track 4.70 -> 8.95 mm
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- added copper zone on B.Cu, net GND
