File: mm_power.kicad_sch (KiCad schematic)
At the start: 1 part, among them J5 Conn_01x02

Commit message: tp2
Parts:
- added C7: 1uF, Capacitor_SMD:C_0603_1608Metric, symbol Device:C
- added C8: 22uF, Capacitor_SMD:C_0603_1608Metric, symbol Device:C
- added D1: LED, LED_SMD:LED_0603_1608Metric, symbol Device:LED
- added R10: 180, Resistor_SMD:R_0603_1608Metric, symbol Device:R
- added U3: LP5907MFX-3.3, Package_TO_SOT_SMD:SOT-23-5, symbol Regulator_Linear:LP5907MFX-3.3
Connections:
- net +BATT: now also C8.1, U3.1 (IN), U3.3 (EN)
- net GND: now also C7.2, C8.2, D1.1 (K), U3.2 (GND)
- new net: D1.2 (A), R10.2
- new net +3V3: C7.1, R10.1, U3.5 (OUT)

Commit message: TP3
Parts:
- C8: value 22uF -> 2.2uF
- C9: renamed from C7; value 1uF -> 2.2uF
- R18: renamed from R10; value 180 -> 330
Changed lines of the file:
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@@
   (symbol (lib_id "Device:C") (at 140.97 77.47 0) (unit 1)
     (in_bom yes) (on_board yes) (dnp no) (fields_autoplaced)
-    (property "Reference" "C7" (at 144.78 76.2 0)
-      (effects (font (size 1.27 1.27)) (justify left))
-    )
-    (property "Value" "1uF" (at 144.78 78.74 0)
+    (property "Reference" "C9" (at 144.78 76.2 0)
+      (effects (font (size 1.27 1.27)) (justify left))
+    )
+    (property "Value" "2.2uF" (at 144.78 78.74 0)
       (effects (font (size 1.27 1.27)) (justify left))
     )
@@
       (project "minimouse"
         (path "/d8fa4cba-2469-4231-847f-065b6b829f44/3f9b0845-5778-418c-a7a8-03da2392145e"
-          (reference "C7") (unit 1)
+          (reference "C9") (unit 1)
         )
       )
@@
   )
   (symbol (lib_id "Device:R") (at 146.05 72.39 90) (unit 1)
-    (in_bom yes) (on_board yes) (dnp no) (fields_autoplaced)
-    (property "Reference" "R10" (at 146.05 66.04 90)
-      (effects (font (size 1.27 1.27)))
-    )
-    (property "Value" "180" (at 146.05 68.58 90)
+    (in_bom yes) (on_board yes) (dnp no)
+    (property "Reference" "R18" (at 146.05 66.04 90)
+      (effects (font (size 1.27 1.27)))
+    )
+    (property "Value" "330" (at 146.05 68.58 90)
       (effects (font (size 1.27 1.27)))
     )
@@
       (project "minimouse"
         (path "/d8fa4cba-2469-4231-847f-065b6b829f44/3f9b0845-5778-418c-a7a8-03da2392145e"
-          (reference "R10") (unit 1)
+          (reference "R18") (unit 1)
         )
       )
@@
       (effects (font (size 1.27 1.27)) (justify left))
     )
-    (property "Value" "22uF" (at 107.95 77.47 0)
-      (effects (font (size 1.27 1.27)) (justify left))
-    )
+    (property "Value" "2.2uF" (at 107.95 77.47 0)
+      (effects (font (size 1.27 1.27)) (justify left))
+    )

Commit message: dernier tp
Connections:
- net +3V3 renamed +3.3V
Other:
- moved on the sheet: C9, D1, J5, R18
